File: kicad-proj/rf-proto-card.kicad_pcb (KiCad board)
At the start: 2 copper layers, 85.6 x 54 mm, 54 parts, among them J1 RF_Shield_One_Piece, J2 sma-a, J3 sma-b, J4 RF_Shield_One_Piece, J5 sma-c, J6 sma-d, U1 GALI-52, U2 GALI-52

Commit message: Updated design and exported gerber
Parts:
- removed FID1: card-info-gold, rf-proto-card:front-info-gold
- removed FID2: card-info-white, rf-proto-card:front-info-white
